Commit message: someone cooked here

File: src/chassis_controls/description/urdf/drive.urdf.xacro (robot description, xacro)
@@ -1,9 +1,9 @@
-<?xml version="1.0"?>
-<robot xmlns:xacro="http://www.ros.org/wiki/xacro" name="drive">
+<?xml version="1.0" encoding="utf-8"?>
+<robot xmlns:xacro="http://www.ros.org/wiki/xacro" name="rover">
     <xacro:arg name="use_gazebo" default="false"/>
-    <xacro:include filename="$(find chassis_controls)/urdf/rmm.urdf" />
+    <xacro:include filename="drive_urdf.urdf" />
     <!-- Import control_xacro -->
     <xacro:include filename="drive_ros2_control.xacro" />
-    <xacro:rmm_ros2_control
+    <xacro:drive_ros2_control
         name="DriveSystem"
         use_gazebo="$(arg use_gazebo)"

File: src/chassis_controls/description/urdf/drive_urdf.urdf (robot description, URDF)
Before this commit: robot rover, 6 links, 6 joints
Links:
- removed link base_footprint
- link FL_wheel: geometry collision mesh filename=package://chassis_controls/description/meshes/visual/FL_whe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; visual mesh filename=package://chassis_controls/description/meshes/visual/FL_whe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
- link FR_wheel: geometry collision mesh filename=package://chassis_controls/description/meshes/visual/FR_whe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; visual mesh filename=package://chassis_controls/description/meshes/visual/FR_whe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
- link RL_wheel: geometry collision mesh filename=package://chassis_controls/description/meshes/visual/RL_whe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; visual mesh filename=package://chassis_controls/description/meshes/visual/RL_whe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
- link RR_wheel: geometry collision mesh filename=package://chassis_controls/description/meshes/visual/RR_whe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; visual mesh filename=package://chassis_controls/description/meshes/visual/RR_whe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
- link base_link: geometry collision mesh filename=package://chassis_controls/description/meshes/visual/base_l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; visual mesh filename=package://chassis_controls/description/meshes/visual/base_l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
Joints:
- removed joint base_footprint_joint
- removed joint base_joint
