Commit message: ready for PID tuning

File: src/chassis_controls/description/urdf/drive_ros2_control.xacro (robot description, xacro)
@@ -9,4 +9,12 @@
                 <xacro:unless value="${use_gazebo}">
                     <plugin>chassis_controls/DriveSystem</plugin>
+                    <param name="wheel_diameter">${wheel_diameter}</param>
+                    <param name="wheel_max_velocity">${wheel_max_velocity}</param>
+                    <param name="wheel_enc_counts_per_rev">${wheel_enc_counts_per_rev}</param>
+                    <param name="controller_period">${controller_period}</param>
+                    <param name="FL_id">${FL_id}</param>
+                    <param name="RR_id">${RR_id}</param>
+                    <param name="FR_id">${FR_id}</param>
+                    <param name="RL_id">${RL_id}</param>
                 </xacro:unless>
             </hardware>

File: src/chassis_controls/description/urdf/rover.urdf.xacro (robot description, xacro)
@@ -2,4 +2,12 @@
 <robot xmlns:xacro="http://www.ros.org/wiki/xacro" name="rover">
     <xacro:arg name="use_gazebo" default="false"/>
+    <xacro:property name="wheel_diameter" value="0.40601"/>
+    <xacro:property name="wheel_max_velocity" value="20.0"/>
+    <xacro:property name="wheel_enc_counts_per_rev" value="1024"/>
+    <xacro:property name="controller_period" value="0.1"/>
+    <xacro:property name="FL_id" value="20"/>
+    <xacro:property name="FR_id" value="10"/>
+    <xacro:property name="RR_id" value="40"/>
+    <xacro:property name="RL_id" value="30"/>
     <xacro:include filename="drive_urdf.urdf" />
     <!-- Import control_xacro -->

Commit message: CIRC 2024

File: src/chassis_controls/description/urdf/drive_ros2_control.xacro (robot description, xacro)
@@ -9,4 +9,5 @@
                 <xacro:unless value="${use_gazebo}">
                     <plugin>chassis_controls/DriveSystem</plugin>
+                    <param name="testing">${testing}</param>
                     <param name="wheel_diameter">${wheel_diameter}</param>
                     <param name="wheel_max_velocity">${wheel_max_velocity}</param>
@@ -17,4 +18,5 @@
                     <param name="FR_id">${FR_id}</param>
                     <param name="RL_id">${RL_id}</param>
+                    <param name="tested_pwm">${tested_pwm}</param>
                 </xacro:unless>
             </hardware>

File: src/chassis_controls/description/urdf/rover.urdf.xacro (robot description, xacro)
@@ -2,4 +2,6 @@
 <robot xmlns:xacro="http://www.ros.org/wiki/xacro" name="rover">
     <xacro:arg name="use_gazebo" default="false"/>
+    <xacro:property name="testing" value="0"/>
+    <xacro:property name="tested_pwm" value="20.0"/>
     <xacro:property name="wheel_diameter" value="0.40601"/>
     <xacro:property name="wheel_max_velocity" value="20.0"/>

Commit message: CIRC gains loaded

File: src/chassis_controls/description/urdf/drive_ros2_control.xacro (robot description, xacro)
@@ -9,4 +9,16 @@
                 <xacro:unless value="${use_gazebo}">
                     <plugin>chassis_controls/DriveSystem</plugin>
+                    <param name="kp_fl">${kp_fl}</param>
+                    <param name="ki_fl">${ki_fl}</param>
+                    <param name="kd_fl">${kd_fl}</param>
+                    <param name="kp_fr">${kp_fr}</param>
+                    <param name="ki_fr">${ki_fr}</param>
+                    <param name="kd_fr">${kd_fr}</param>
+                    <param name="kp_rl">${kp_rl}</param>
+                    <param name="ki_rl">${ki_rl}</param>
+                    <param name="kd_rl">${kd_rl}</param>
+                    <param name="kp_rr">${kp_rr}</param>
+                    <param name="ki_rr">${ki_rr}</param>
+                    <param name="kd_rr">${kd_rr}</param>
                     <param name="testing">${testing}</param>
                     <param name="wheel_diameter">${wheel_diameter}</param>

File: src/chassis_controls/description/urdf/rover.urdf.xacro (robot description, xacro)
@@ -2,4 +2,16 @@
 <robot xmlns:xacro="http://www.ros.org/wiki/xacro" name="rover">
     <xacro:arg name="use_gazebo" default="false"/>
+    <xacro:property name="kp_fl" value="0.7322"/>
+    <xacro:property name="ki_fl" value="1.1277"/>
+    <xacro:property name="kd_fl" value="0.0"/>
+    <xacro:property name="kp_fr" value="0.9078"/>
+    <xacro:property name="ki_fr" value="1.495"/>
+    <xacro:property name="kd_fr" value="0"/>
+    <xacro:property name="kp_rl" value="0.7232"/>
+    <xacro:property name="ki_rl" value="1.13"/>
+    <xacro:property name="kd_rl" value="0"/>
+    <xacro:property name="kp_rr" value="1.041"/>
+    <xacro:property name="ki_rr" value="1.114"/>
+    <xacro:property name="kd_rr" value="0"/>
     <xacro:property name="testing" value="0"/>
     <xacro:property name="tested_pwm" value="20.0"/>
@@ -8,8 +20,8 @@
     <xacro:property name="wheel_enc_counts_per_rev" value="4096"/>
     <xacro:property name="controller_period" value="0.1"/>
-    <xacro:property name="FL_id" value="30"/>
-    <xacro:property name="FR_id" value="40"/>
-    <xacro:property name="RR_id" value="10"/>
-    <xacro:property name="RL_id" value="20"/>
+    <xacro:property name="FL_id" value="10"/>
+    <xacro:property name="FR_id" value="30"/>
+    <xacro:property name="RR_id" value="20"/>
+    <xacro:property name="RL_id" value="40"/>
     <xacro:include filename="drive_urdf.urdf" />
     <!-- Import control_xacro -->

Commit message: Improve drive code. Clean up repository.

File: src/chassis_controls/description/urdf/drive_ros2_control.xacro (robot description, xacro)
@@ -9,26 +9,22 @@
                 <xacro:unless value="${use_gazebo}">
                     <plugin>chassis_controls/DriveSystem</plugin>
-                    <param name="kp_fl">${kp_fl}</param>
-                    <param name="ki_fl">${ki_fl}</param>
-                    <param name="kd_fl">${kd_fl}</param>
-                    <param name="kp_fr">${kp_fr}</param>
-                    <param name="ki_fr">${ki_fr}</param>
-                    <param name="kd_fr">${kd_fr}</param>
-                    <param name="kp_rl">${kp_rl}</param>
-                    <param name="ki_rl">${ki_rl}</param>
-                    <param name="kd_rl">${kd_rl}</param>
-                    <param name="kp_rr">${kp_rr}</param>
-                    <param name="ki_rr">${ki_rr}</param>
-                    <param name="kd_rr">${kd_rr}</param>
-                    <param name="testing">${testing}</param>
+                    <param name="FL_id">${FL_id}</param>
+                    <param name="FR_id">${FR_id}</param>
+                    <param name="RR_id">${RR_id}</param>
+                    <param name="RL_id">${RL_id}</param>
+                    <param name="Kp_FL">${Kp_FL}</param>
+                    <param name="Ki_FL">${Ki_FL}</param>
+                    <param name="Kd_FL">${Kd_FL}</param>
+                    <param name="Kp_FR">${Kp_FR}</param>
+                    <param name="Ki_FR">${Ki_FR}</param>
+                    <param name="Kd_FR">${Kd_FR}</param>
+                    <param name="Kp_RR">${Kp_RR}</param>
+                    <param name="Ki_RR">${Ki_RR}</param>
+                    <param name="Kd_RR">${Kd_RR}</param>
+                    <param name="Kp_RL">${Kp_RL}</param>
+                    <param name="Ki_RL">${Ki_RL}</param>
+                    <param name="Kd_RL">${Kd_RL}</param>
                     <param name="wheel_diameter">${wheel_diameter}</param>
-                    <param name="wheel_max_velocity">${wheel_max_velocity}</param>
-                    <param name="wheel_enc_counts_per_rev">${wheel_enc_counts_per_rev}</param>
-                    <param name="controller_period">${controller_period}</param>
-                    <param name="FL_id">${FL_id}</param>
-                    <param name="RR_id">${RR_id}</param>
-                    <param name="FR_id">${FR_id}</param>
-                    <param name="RL_id">${RL_id}</param>
-                    <param name="tested_pwm">${tested_pwm}</param>
+                    <param name="wheel_encoder_counts_per_revolution">${wheel_encoder_counts_per_revolution}</param>
                 </xacro:unless>
             </hardware>
@@ -38,6 +34,6 @@
                     <param name="max">10</param>
                 </command_interface>
+                <state_interface name="position" />
                 <state_interface name="velocity" />
-                <state_interface name="position" />
             </joint>
             <joint name="q2"> <!-- FR_wheel -->
@@ -46,6 +42,6 @@
                     <param name="max">10</param>
                 </command_interface>
+                <state_interface name="position" />
                 <state_interface name="velocity" />
-                <state_interface name="position" />
             </joint>
             <joint name="q3"> <!-- RR_wheel -->
@@ -54,6 +50,6 @@
                     <param name="max">10</param>
                 </command_interface>
+                <state_interface name="position" />
                 <state_interface name="velocity" />
-                <state_interface name="position" />
             </joint>
             <joint name="q4"> <!-- RL_wheel -->
@@ -62,6 +58,6 @@
                     <param name="max">10</param>
                 </command_interface>
+                <state_interface name="position" />
                 <state_interface name="velocity" />
-                <state_interface name="position" />
             </joint>
         </ros2_control>

File: src/chassis_controls/description/urdf/rover.urdf.xacro (robot description, xacro)
@@ -2,26 +2,22 @@
 <robot xmlns:xacro="http://www.ros.org/wiki/xacro" name="rover">
     <xacro:arg name="use_gazebo" default="false"/>
-    <xacro:property name="kp_fl" value="1.7322"/>
-    <xacro:property name="ki_fl" value="1.1277"/>
-    <xacro:property name="kd_fl" value="0.0"/>
-    <xacro:property name="kp_fr" value="1.9078"/>
-    <xacro:property name="ki_fr" value="1.495"/>
-    <xacro:property name="kd_fr" value="0"/>
-    <xacro:property name="kp_rl" value="1.7232"/>
-    <xacro:property name="ki_rl" value="1.13"/>
-    <xacro:property name="kd_rl" value="0"/>
-    <xacro:property name="kp_rr" value="1.941"/>
-    <xacro:property name="ki_rr" value="1.114"/>
-    <xacro:property name="kd_rr" value="0"/>
-    <xacro:property name="testing" value="0"/>
-    <xacro:property name="tested_pwm" value="20.0"/>
+    <xacro:property name="FL_id" value="20"/>
+    <xacro:property name="FR_id" value="40"/>
+    <xacro:property name="RR_id" value="10"/>
+    <xacro:property name="RL_id" value="30"/>
+    <xacro:property name="Kp_FL" value="0.4"/>
+    <xacro:property name="Ki_FL" value="0.002"/>
+    <xacro:property name="Kd_FL" value="160.0"/>
+    <xacro:property name="Kp_FR" value="0.4"/>
+    <xacro:property name="Ki_FR" value="0.002"/>
+    <xacro:property name="Kd_FR" value="160.0"/>
+    <xacro:property name="Kp_RR" value="0.4"/>
+    <xacro:property name="Ki_RR" value="0.002"/>
+    <xacro:property name="Kd_RR" value="160.0"/>
+    <xacro:property name="Kp_RL" value="0.4"/>
+    <xacro:property name="Ki_RL" value="0.002"/>
+    <xacro:property name="Kd_RL" value="160.0"/>
     <xacro:property name="wheel_diameter" value="0.40601"/>
-    <xacro:property name="wheel_max_velocity" value="20.0"/>
-    <xacro:property name="wheel_enc_counts_per_rev" value="4096"/>
-    <xacro:property name="controller_period" value="0.1"/>
-    <xacro:property name="FL_id" value="10"/>
-    <xacro:property name="FR_id" value="30"/>
-    <xacro:property name="RR_id" value="20"/>
-    <xacro:property name="RL_id" value="40"/>
+    <xacro:property name="wheel_encoder_counts_per_revolution" value="4096"/>
     <xacro:include filename="drive_urdf.urdf" />
     <!-- Import control_xacro -->

Commit message: Adding open loop drive system. Improving modularity of existing source code and cleaning it up

File: src/chassis_controls/description/urdf/drive_ros2_control.xacro (robot description, xacro)
@@ -1,5 +1,5 @@
 <?xml version="1.0" encoding="utf-8"?>
 <robot xmlns:xacro="http://www.ros.org/wiki/xacro">
-    <xacro:macro name="drive_ros2_control" params="name use_gazebo">
+    <xacro:macro name="drive_ros2_control" params="name use_gazebo open_loop">
         <ros2_control name="${name}" type="system">
             <hardware>
@@ -8,23 +8,34 @@
                 </xacro:if>
                 <xacro:unless value="${use_gazebo}">
-                    <plugin>chassis_controls/DriveSystem</plugin>
-                    <param name="FL_id">${FL_id}</param>
-                    <param name="FR_id">${FR_id}</param>
-                    <param name="RR_id">${RR_id}</param>
-                    <param name="RL_id">${RL_id}</param>
-                    <param name="Kp_FL">${Kp_FL}</param>
-                    <param name="Ki_FL">${Ki_FL}</param>
-                    <param name="Kd_FL">${Kd_FL}</param>
-                    <param name="Kp_FR">${Kp_FR}</param>
-                    <param name="Ki_FR">${Ki_FR}</param>
-                    <param name="Kd_FR">${Kd_FR}</param>
-                    <param name="Kp_RR">${Kp_RR}</param>
-                    <param name="Ki_RR">${Ki_RR}</param>
-                    <param name="Kd_RR">${Kd_RR}</param>
-                    <param name="Kp_RL">${Kp_RL}</param>
-                    <param name="Ki_RL">${Ki_RL}</param>
-                    <param name="Kd_RL">${Kd_RL}</param>
-                    <param name="wheel_diameter">${wheel_diameter}</param>
-                    <param name="wheel_encoder_counts_per_revolution">${wheel_encoder_counts_per_revolution}</param>
+                    <xacro:if value="${open_loop}">
+                        <plugin>chassis_controls/DriveSystemOpenLoop</plugin>
+                        <param name="FL_id">${FL_id}</param>
+                        <param name="FR_id">${FR_id}</param>
+                        <param name="RR_id">${RR_id}</param>
+                        <param name="RL_id">${RL_id}</param>
+                        <param name="wheel_diameter">${wheel_diameter}</param>
+                        <param name="max_wheel_rad_per_sec">${max_wheel_rad_per_sec}</param>
+                    </xacro:if>
+                    <xacro:unless value="${open_loop}">
+                        <plugin>chassis_controls/DriveSystem</plugin>
+                        <param name="FL_id">${FL_id}</param>
+                        <param name="FR_id">${FR_id}</param>
+                        <param name="RR_id">${RR_id}</param>
+                        <param name="RL_id">${RL_id}</param>
+                        <param name="Kp_FL">${Kp_FL}</param>
+                        <param name="Ki_FL">${Ki_FL}</param>
+                        <param name="Kd_FL">${Kd_FL}</param>
+                        <param name="Kp_FR">${Kp_FR}</param>
+                        <param name="Ki_FR">${Ki_FR}</param>
+                        <param name="Kd_FR">${Kd_FR}</param>
+                        <param name="Kp_RR">${Kp_RR}</param>
+                        <param name="Ki_RR">${Ki_RR}</param>
+                        <param name="Kd_RR">${Kd_RR}</param>
+                        <param name="Kp_RL">${Kp_RL}</param>
+                        <param name="Ki_RL">${Ki_RL}</param>
+                        <param name="Kd_RL">${Kd_RL}</param>
+                        <param name="wheel_diameter">${wheel_diameter}</param>
+                        <param name="wheel_encoder_counts_per_revolution">${wheel_encoder_counts_per_revolution}</param>
+                    </xacro:unless>
                 </xacro:unless>
             </hardware>

File: src/chassis_controls/description/urdf/rover.urdf.xacro (robot description, xacro)
@@ -3,4 +3,5 @@
     <xacro:arg name="use_gazebo" default="false"/>
     <xacro:arg name="sport_mode" default="true"/>
+    <xacro:arg name="open_loop" default="false"/>
     <xacro:property name="FL_id" value="20"/>
     <xacro:property name="FR_id" value="40"/>
@@ -39,4 +40,5 @@
     <xacro:property name="wheel_diameter" value="0.40601"/>
     <xacro:property name="wheel_encoder_counts_per_revolution" value="4096"/>
+    <xacro:property name="max_wheel_rad_per_sec" value="10.0"/>
     <xacro:include filename="drive_urdf.urdf" />
     <!-- Import control_xacro -->
