Commit message: sorted out CAN ids (again)

File: src/chassis_controls/description/urdf/rover.urdf.xacro (robot description, xacro)
@@ -7,6 +7,6 @@
     <xacro:property name="controller_period" value="0.1"/>
     <xacro:property name="FL_id" value="20"/>
-    <xacro:property name="FR_id" value="10"/>
-    <xacro:property name="RR_id" value="40"/>
+    <xacro:property name="FR_id" value="40"/>
+    <xacro:property name="RR_id" value="10"/>
     <xacro:property name="RL_id" value="30"/>
     <xacro:include filename="drive_urdf.urdf" />

Commit message: testing done

File: src/chassis_controls/description/urdf/rover.urdf.xacro (robot description, xacro)
@@ -4,10 +4,10 @@
     <xacro:property name="wheel_diameter" value="0.40601"/>
     <xacro:property name="wheel_max_velocity" value="20.0"/>
-    <xacro:property name="wheel_enc_counts_per_rev" value="1024"/>
+    <xacro:property name="wheel_enc_counts_per_rev" value="4096"/>
     <xacro:property name="controller_period" value="0.1"/>
-    <xacro:property name="FL_id" value="20"/>
+    <xacro:property name="FL_id" value="30"/>
     <xacro:property name="FR_id" value="40"/>
     <xacro:property name="RR_id" value="10"/>
-    <xacro:property name="RL_id" value="30"/>
+    <xacro:property name="RL_id" value="20"/>
     <xacro:include filename="drive_urdf.urdf" />
     <!-- Import control_xacro -->

Commit message: arm dexterity mission v1

File: src/chassis_controls/description/urdf/rover.urdf.xacro (robot description, xacro)
@@ -2,14 +2,14 @@
 <robot xmlns:xacro="http://www.ros.org/wiki/xacro" name="rover">
     <xacro:arg name="use_gazebo" default="false"/>
-    <xacro:property name="kp_fl" value="0.7322"/>
+    <xacro:property name="kp_fl" value="1.7322"/>
     <xacro:property name="ki_fl" value="1.1277"/>
     <xacro:property name="kd_fl" value="0.0"/>
-    <xacro:property name="kp_fr" value="0.9078"/>
+    <xacro:property name="kp_fr" value="1.9078"/>
     <xacro:property name="ki_fr" value="1.495"/>
     <xacro:property name="kd_fr" value="0"/>
-    <xacro:property name="kp_rl" value="0.7232"/>
+    <xacro:property name="kp_rl" value="1.7232"/>
     <xacro:property name="ki_rl" value="1.13"/>
     <xacro:property name="kd_rl" value="0"/>
-    <xacro:property name="kp_rr" value="1.041"/>
+    <xacro:property name="kp_rr" value="1.941"/>
     <xacro:property name="ki_rr" value="1.114"/>
     <xacro:property name="kd_rr" value="0"/>

Commit message: Drive fine tuning

File: src/chassis_controls/description/urdf/rover.urdf.xacro (robot description, xacro)
@@ -2,20 +2,39 @@
 <robot xmlns:xacro="http://www.ros.org/wiki/xacro" name="rover">
     <xacro:arg name="use_gazebo" default="false"/>
+    <xacro:arg name="sport_mode" default="true"/>
     <xacro:property name="FL_id" value="20"/>
     <xacro:property name="FR_id" value="40"/>
     <xacro:property name="RR_id" value="10"/>
     <xacro:property name="RL_id" value="30"/>
-    <xacro:property name="Kp_FL" value="0.4"/>
-    <xacro:property name="Ki_FL" value="0.002"/>
-    <xacro:property name="Kd_FL" value="160.0"/>
-    <xacro:property name="Kp_FR" value="0.4"/>
-    <xacro:property name="Ki_FR" value="0.002"/>
-    <xacro:property name="Kd_FR" value="160.0"/>
-    <xacro:property name="Kp_RR" value="0.4"/>
-    <xacro:property name="Ki_RR" value="0.002"/>
-    <xacro:property name="Kd_RR" value="160.0"/>
-    <xacro:property name="Kp_RL" value="0.4"/>
-    <xacro:property name="Ki_RL" value="0.002"/>
-    <xacro:property name="Kd_RL" value="160.0"/>
+    <!-- Allow for different PID gains to be used to select between
+    acceleration/responsivness and power usage -->
+    <xacro:if value="$(arg sport_mode)">
+        <xacro:property name="Kp_FL" value="0.8"/>
+        <xacro:property name="Ki_FL" value="0.008"/>
+        <xacro:property name="Kd_FL" value="220.0"/>
+        <xacro:property name="Kp_FR" value="0.8"/>
+        <xacro:property name="Ki_FR" value="0.008"/>
+        <xacro:property name="Kd_FR" value="220.0"/>
+        <xacro:property name="Kp_RR" value="0.8"/>
+        <xacro:property name="Ki_RR" value="0.008"/>
+        <xacro:property name="Kd_RR" value="220.0"/>
+        <xacro:property name="Kp_RL" value="0.8"/>
+        <xacro:property name="Ki_RL" value="0.008"/>
+        <xacro:property name="Kd_RL" value="220.0"/>
+    </xacro:if>
+    <xacro:unless value="$(arg sport_mode)">
+        <xacro:property name="Kp_FL" value="0.4"/>
+        <xacro:property name="Ki_FL" value="0.002"/>
+        <xacro:property name="Kd_FL" value="160.0"/>
+        <xacro:property name="Kp_FR" value="0.4"/>
+        <xacro:property name="Ki_FR" value="0.002"/>
+        <xacro:property name="Kd_FR" value="160.0"/>
+        <xacro:property name="Kp_RR" value="0.4"/>
+        <xacro:property name="Ki_RR" value="0.002"/>
+        <xacro:property name="Kd_RR" value="160.0"/>
+        <xacro:property name="Kp_RL" value="0.4"/>
+        <xacro:property name="Ki_RL" value="0.002"/>
+        <xacro:property name="Kd_RL" value="160.0"/>
+    </xacro:unless>
     <xacro:property name="wheel_diameter" value="0.40601"/>
     <xacro:property name="wheel_encoder_counts_per_revolution" value="4096"/>

Commit message: Initial autonav mvp files

File: src/chassis_controls/description/urdf/rover.urdf.xacro (robot description, xacro)
@@ -46,3 +46,62 @@
         use_gazebo="$(arg use_gazebo)"
     />
+    <link name="base_footprint">
+    </link>
+    <joint name="base_footprint_joint" type="fixed">
+        <parent link="base_link" />
+        <child link="base_footprint" />
+        <origin xyz="0 0 0" rpy="0 0 0" />
+    </joint>
+    <xacro:macro name="box_inertia" params="m w h d">
+        <inertial>
+            <origin xyz="0 0 0" rpy="${pi/2} 0 ${pi/2}" />
+            <mass value="${m}" />
+            <inertia ixx="${(m/12) * (h*h + d*d)}" ixy="0.0" ixz="0.0" iyy="${(m/12) * (w*w + d*d)}"
+                iyz="0.0" izz="${(m/12) * (w*w + h*h)}" />
+        </inertial>
+    </xacro:macro>
+    <link name="imu_link">
+        <visual>
+            <origin xyz="0 0 0" rpy="0 0 0" />
+            <geometry>
+                <box size="0.025 0.025 0.025" />
+            </geometry>
+        </visual>
+        <collision>
+            <origin xyz="0 0 0" rpy="0 0 0" />
+            <geometry>
+                <box size="0.025 0.025 0.025" />
+            </geometry>
+        </collision>
+        <xacro:box_inertia m="0.1" w="0.1" d="0.1" h="0.1" />
+    </link>
+    <joint name="imu_joint" type="fixed">
+        <parent link="base_link" />
+        <child link="imu_link" />
+        <origin xyz="0 0 0.25" />
+    </joint>
+    <link name="lidar_link">
+        <inertial>
+            <origin xyz="0 0 0" rpy="0 0 0" />
+            <mass value="0.125" />
+            <inertia ixx="0.001" ixy="0" ixz="0" iyy="0.001" iyz="0" izz="0.001" />
+        </inertial>
+        <collision>
+            <origin xyz="0 0 0" rpy="0 0 0" />
+            <geometry>
+                <cylinder radius="0.0508" length="0.055" />
+            </geometry>
+        </collision>
+        <visual>
+            <origin xyz="0 0 0" rpy="0 0 0" />
+            <geometry>
+                <cylinder radius="0.0508" length="0.055" />
+            </geometry>
+        </visual>
+    </link>
+    <joint name="lidar_joint" type="fixed">
+        <parent link="base_link" />
+        <child link="lidar_link" />
+        <origin xyz="0 0 0.45" rpy="0 0 0" />
+    </joint>
 </robot>

Commit message: Adding april tag pose detection

File: src/chassis_controls/description/urdf/rover.urdf.xacro (robot description, xacro)
@@ -105,3 +105,23 @@
         <origin xyz="0 0 0.45" rpy="0 0 0" />
     </joint>
+    <link name="camera">
+        <visual>
+            <origin xyz="0 0 0" rpy="0 0 0" />
+            <geometry>
+                <box size="0.025 0.025 0.025" />
+            </geometry>
+        </visual>
+        <collision>
+            <origin xyz="0 0 0" rpy="0 0 0" />
+            <geometry>
+                <box size="0.025 0.025 0.025" />
+            </geometry>
+        </collision>
+        <xacro:box_inertia m="0.1" w="0.1" d="0.1" h="0.1" />
+    </link>
+    <joint name="camera_joint" type="fixed">
+        <parent link="base_link" />
+        <child link="camera" />
+        <origin xyz="-0.36 0.24 0.92" rpy="${-pi/2} 0 ${-pi/2}" />
+    </joint>
 </robot>
