Commit message: rover arm and end effector moveit configurations created in src/arm_moveit_config

File: src/arm_urdf/urdf/uorover_ik_urdf.urdf (robot description, URDF)
Before this commit: robot uorover_ik_urdf, 8 links, 7 joints
Joints:
- joint base_footprint_joint: child L1 -> base_footprint; parent base_footprint -> L1
- joint q1: limit lower=0 upper=0 effort=0 velocity=0 -> lower=-3.1415 upper=3.1415 effort=0 velocity=0
- joint q2: limit lower=0 upper=0 effort=0 velocity=0 -> lower=-3.1415 upper=3.1415 effort=0 velocity=0
- joint q3: limit lower=0 upper=0 effort=0 velocity=0 -> lower=-3.1415 upper=3.1415 effort=0 velocity=0
- joint q4: limit lower=0 upper=0 effort=0 velocity=0 -> lower=-3.1415 upper=3.1415 effort=0 velocity=0
- joint q6: limit lower=0 upper=0 effort=0 velocity=0 -> lower=-3.1415 upper=3.1415 effort=0 velocity=0

Commit message: cartesian servo working demo, see issue 91 for video

File: src/arm_urdf/urdf/uorover_ik_urdf.urdf (robot description, URDF)
Before this commit: robot uorover_ik_urdf, 8 links, 7 joints
Joints:
- joint base_footprint_joint: child base_footprint -> L1; parent L1 -> base_footprint
